File: StarLight.kicad_pcb (KiCad board)
At the start: 2 copper layers, 94.3 x 91.6 mm, 18 parts, among them J1 Conn_01x02_Socket, U1 NE555P, U2 4017

Commit message: BRO.
how about you tell me BEFORE I SOLDER EVERYTHING ONTO THE BOARD THAT I MADE A MISTAKE OHH MY DAYS BRO OH MY DAYS. GENUINELY. TS BOARD IS RAGEBAITING?? I CANT
Parts:
- U2: footprint footprints1:N16 -> footprints:N16
Routing:
- net TR: track 69.1 -> 85.2 mm, vias 0 -> 1
- net Net-(D1-K): track 246.5 -> 248.0 mm
- net Net-(D1-A): track 49.6 -> 50.3 mm
Other:
- board text added: "('｡• ᵕ •｡`) <3"
- board text added: "(≧◡≦)"
- board text added: "所到之处皆为光"
