File: StarLight.kicad_sch (KiCad schematic)
At the start: 18 parts, among them J1 Conn_01x02_Socket, U1 NE555P, U2 4017

Commit message: BRO.
how about you tell me BEFORE I SOLDER EVERYTHING ONTO THE BOARD THAT I MADE A MISTAKE OHH MY DAYS BRO OH MY DAYS. GENUINELY. TS BOARD IS RAGEBAITING?? I CANT
Parts:
- U2: footprint footprints1:N16 -> footprints:N16
Changed lines of the file:
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@@
 			)
 		)
-		(property "Footprint" "footprints1:N16"
+		(property "Footprint" "footprints:N16"
 			(at 114.3 41.91 0)
 			(effects
