File: StarLight/StarLight.kicad_pcb (KiCad board)
At the start: 2 copper layers, 92.4 x 89.9 mm, 20 parts, among them J1 Conn_01x02_Socket, U1 NE555P, U2 4017

Commit message: NEW GERBERS
this better be right or im gonna lose it. this is my last time ordering the pcb if it fails this time too i will do unspeakable things
Parts:
- removed G*** (x2): LOGO, LOGO
- U2: footprint cd4017:N16 -> footprints1:N16
Connections:
- R1 pad 2: Net-(U1-DISCH) -> TR
- RV1 pad 1: Net-(U1-DISCH) -> TR
- RV1 pad 2: Net-(U1-DISCH) -> TR
- U1 pad 7: Net-(U1-DISCH) -> TR
Routing:
- net Net-(U1-DISCH): track 35.7 -> 0.00 mm
- net TR: track 39.2 -> 69.1 mm, vias 1 -> 0
- net Net-(D1-K): track 247.9 -> 246.5 mm
- net Net-(D1-A): track 50.5 -> 49.6 mm
- net Net-(D3-A): track 27.8 -> 28.5 mm
Other:
- board size 92.4 x 89.9 mm -> 94.3 x 91.6 mm
- board text removed: "('｡• ᵕ •｡`) <3"
- board text removed: "(≧◡≦)"
- board text removed: "+"
- board text removed: "made with <3 by sua shoot for the stars"
